File: pcb/so-dimm-debugger-programmer.kicad_pcb (KiCad board)
At the start: 2 copper layers, 48.9 x 131.2 mm, 51 parts, among them J1 1612618-4, J10 DNP, J12 Conn_01x06_Pin, J13 DNP, J2 Conn_01x06_Pin, J3 Conn_01x04_Pin, J4 Conn_01x04_Pin, J5 DNP, J6 USB4105-GF-A, J7 USB4105-GF-A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

Commit message: small pcb changes?
Routing:
- net GND: track 18.1 -> 17.4 mm, vias 29 -> 28
Changed lines of the file:
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@@
   (segment (start 134.560205 75.036547) (end 135.710205 76.186547) (width 0.2) (layer "F.Cu") (net 22))
   (segment (start 131.118205 85.965547) (end 131.118205 76.372201) (width 0.2) (layer "F.Cu") (net 22))
-  (segment (start 118.872 108.475547) (end 120.100205 108.475547) (width 0.2) (layer "F.Cu") (net 22))
+  (segment (start 118.635547 108.475547) (end 120.100205 108.475547) (width 0.2) (layer "F.Cu") (net 22))
+  (segment (start 118.618 108.458) (end 118.635547 108.475547) (width 0.2) (layer "F.Cu") (net 22))
   (segment (start 129.213205 87.870547) (end 131.118205 85.965547) (width 0.2) (layer "F.Cu") (net 22))
   (segment (start 131.118205 76.372201) (end 132.453859 75.036547) (width 0.2) (layer "F.Cu") (net 22))
   (via (at 129.213205 87.870547) (size 0.6) (drill 0.3) (layers "F.Cu" "B.Cu") (net 22))
-  (via (at 118.872 108.475547) (size 0.5) (drill 0.3) (layers "F.Cu" "B.Cu") (net 22))
-  (segment (start 118.364 107.967547) (end 118.364 105.069752) (width 0.2) (layer "B.Cu") (net 22))
+  (via (at 118.618 108.458) (size 0.5) (drill 0.3) (layers "F.Cu" "B.Cu") (net 22))
+  (segment (start 122.355205 92.696547) (end 127.181205 87.870547) (width 0.2) (layer "B.Cu") (net 22))
+  (segment (start 118.618 108.458) (end 118.364 108.204) (width 0.2) (layer "B.Cu") (net 22))
   (segment (start 127.181205 87.870547) (end 129.213205 87.870547) (width 0.2) (layer "B.Cu") (net 22))
+  (segment (start 118.364 105.069752) (end 122.355205 101.078547) (width 0.2) (layer "B.Cu") (net 22))
   (segment (start 122.355205 101.078547) (end 122.355205 92.696547) (width 0.2) (layer "B.Cu") (net 22))
-  (segment (start 118.872 108.475547) (end 118.364 107.967547) (width 0.2) (layer "B.Cu") (net 22))
-  (segment (start 122.355205 92.696547) (end 127.181205 87.870547) (width 0.2) (layer "B.Cu") (net 22))
-  (segment (start 118.364 105.069752) (end 122.355205 101.078547) (width 0.2) (layer "B.Cu") (net 22))
+  (segment (start 118.364 108.204) (end 118.364 105.069752) (width 0.2) (layer "B.Cu") (net 22))
   (segment (start 126.106053 101.071547) (end 129.841205 101.071547) (width 0.2) (layer "F.Cu") (net 24))
   (segment (start 129.841205 101.071547) (end 129.848205 101.078547) (width 0.2) (layer "F.Cu") (net 24))
@@
   (segment (start 122.096205 119.117547) (end 126.673205 114.540547) (width 0.5) (layer "B.Cu") (net 174))
   (segment (start 104.550205 162.3516) (end 104.550205 161.2896) (width 0.25) (layer "F.Cu") (net 175))
+  (segment (start 107.250205 148.949547) (end 107.250205 150.899547) (width 0.25) (layer "F.Cu") (net 175))
   (segment (start 114.634205 155.561547) (end 114.989205 155.561547) (width 0.5) (layer "F.Cu") (net 175))
   (segment (start 124.3588 161.3412) (end 124.1552 161.1376) (width 0.25) (layer "F.Cu") (net 175))
@@
   (segment (start 127.688205 159.026547) (end 127.688205 160.005547) (width 0.2) (layer "F.Cu") (net 175))
   (segment (start 119.548205 138.162547) (end 118.799205 138.162547) (width 0.5) (layer "F.Cu") (net 175))
-  (segment (start 107.250205 148.949547) (end 107.750205 148.449547) (width 0.25) (layer "F.Cu") (net 175))
   (segment (start 114.989205 155.561547) (end 115.497205 155.053547) (width 0.5) (layer "F.Cu") (net 175))
   (segment (start 110.950205 162.013547) (end 111.052205 161.911547) (width 0.25) (layer "F.Cu") (net 175))
   (segment (start 130.7588 162.2246) (end 130.7588 161.7476) (width 0.25) (layer "F.Cu") (net 175))
   (segment (start 124.3588 162.2246) (end 124.3588 161.3412) (width 0.25) (layer "F.Cu") (net 175))
-  (segment (start 107.250205 150.899547) (end 107.250205 148.949547) (width 0.25) (layer "F.Cu") (net 175))
   (segment (start 107.750205 159.280547) (end 107.750205 160.006547) (width 0.2) (layer "F.Cu") (net 175))
   (segment (start 120.196205 133.977047) (end 120.196205 132.714547) (width 0.5) (layer "F.Cu") (net 175))
@@
   (via (at 118.418205 138.543547) (size 0.8) (drill 0.4) (layers "F.Cu" "B.Cu") (net 175))
   (via (at 106.099205 154.164547) (size 0.6) (drill 0.3) (layers "F.Cu" "B.Cu") (free) (net 175))
-  (via (at 107.750205 148.449547) (size 0.6) (drill 0.3) (layers "F.Cu" "B.Cu") (net 175))
   (via (at 111.052205 155.434547) (size 0.6) (drill 0.3) (layers "F.Cu" "B.Cu") (free) (net 175))
   (via (at 106.861205 152.640547) (size 0.6) (drill 0.3) (layers "F.Cu" "B.Cu") (net 175))
